Commit message: add some drivers

File: src/simulation/robot/spot_description/urdf/accessories.urdf.xacro (robot description, xacro)
@@ -1,68 +1,77 @@
 <?xml version="1.0"?>
-<robot xmlns:xacro="http://ros.org/wiki/xacro">
-    <xacro:property name="M_PI" value="3.1415926535897931" />
-    <xacro:include filename="$(find spot_description)/urdf/constants.urdf.xacro" />
-    <xacro:include filename="$(find spot_description)/urdf/asus_camera.urdf.xacro" />
-    <xacro:include filename="$(find spot_description)/urdf/generic_stereo_camera.urdf.xacro" />
-    <!--
-    <xacro:asus_camera parent="base_link" name="camera">
-        <origin xyz="${base_length / 2} 0.0 ${base_height / 2 - 0.01}" rpy="0 ${M_PI/12} 0"/>
-    </xacro:asus_camera>
-    <xacro:generic_stereo_camera parent="base_link" name="stereo_camera" ros_topic="image_raw" cam_info_topic="camera_info"
-                                 update_rate="30" height="480" width="640" image_format="R8G8B8" hfov="2.094395102" baseline="0.08" focal_length="184.7520861">
-        <origin xyz="${base_length / 2} 0.0 ${base_height / 2 - 0.01}" rpy="0 ${M_PI/12} 0"/>
-    </xacro:generic_stereo_camera>
-    -->
-    <gazebo>
-        <plugin name="imu_controller" filename="libhector_gazebo_ros_imu.so">
-            <updateRate>50.0</updateRate>
-            <bodyName>imu_link</bodyName>
-            <topicName>imu/data</topicName>
-            <accelDrift>0.005 0.005 0.005</accelDrift>
-            <accelGaussianNoise>0.005 0.005 0.005</accelGaussianNoise>
-            <rateDrift>0.005 0.005 0.005 </rateDrift>
-            <rateGaussianNoise>0.005 0.005 0.005 </rateGaussianNoise>
-            <headingDrift>0.005</headingDrift>
-            <headingGaussianNoise>0.005</headingGaussianNoise>
-        </plugin>
-    </gazebo>
-    <link name="imu_link">
-        <inertial>
-            <mass value="0.001"/>
-            <origin xyz="0 0 0" rpy="0 0 0"/>
-            <inertia ixx="1e-09" ixy="0.0" ixz="0.0" iyy="1e-09" iyz="0.0" izz="1e-09"/>
-        </inertial>
+<robot xmlns:xacro="http://www.ros.org/wiki/xacro">
+  <xacro:if value="$(optenv SPOT_PACK 0)">
+    <joint name="pack_mount_joint" type="fixed">
+      <parent link="base_link"/>
+      <child link="pack_mount"/>
+      <origin xyz="-0.019986 0 0.093662" rpy="0 0 0"/>
+    </joint>
+    <link name="pack_mount">
+      <visual>
+        <geometry>
+          <mesh filename="package://spot_description/meshes/pack_top.dae"/>
+        </geometry>
+      </visual>
+      <visual>
+        <geometry>
+          <mesh filename="package://spot_description/meshes/pack_body.dae"/>
+        </geometry>
+      </visual>
+      <collision>
+        <geometry>
+          <mesh filename="package://spot_description/meshes/pack_body.dae"/>
+        </geometry>
+      </collision>
     </link>
-    <joint name="imu_joint" type="fixed">
-        <parent link="base_link" />
-        <child link="imu_link" />
+  </xacro:if>
+  <xacro:if value="$(optenv SPOT_LIDAR_MOUNT 0)">
+    <joint name="lidar_mount_joint" type="fixed">
+      <parent link="pack_mount"/>
+      <child link="lidar_mount"/>
+      <origin xyz="0.015 0 0.149285" rpy="0 0 0"/>
     </joint>
-    <!-- <xacro:include filename="$(find velodyne_description)/urdf/VLP-16.urdf.xacro"/>
-    <xacro:VLP-16 parent="base_link" name="velodyne" topic="velodyne_points" hz="10" samples="1024" gpu="false" lasers="16" max_range="100">
-        <origin xyz="0.29 0 ${(base_height / 2) - 0.01}" rpy="0 0 0" />
-    </xacro:VLP-16> -->
-    <link name="camera_link">
+    <link name="lidar_mount">
+      <visual>
+        <geometry>
+          <mesh filename="package://spot_description/meshes/lidar_mount.dae"/>
+        </geometry>
+      </visual>
+      <collision>
+        <geometry>
+          <mesh filename="package://spot_description/meshes/lidar_mount_collision.stl"/>
+        </geometry>
+      </collision>
     </link>
-    <joint name="camera_joint" type="fixed">
-        <parent link="link06" />
-        <child link="camera_link" />
-    </joint>
-    <xacro:generic_stereo_camera parent="camera_link" name="stereo_camera" ros_topic="image_raw" cam_info_topic="camera_info"
-                                 update_rate="30" height="480" width="640" image_format="R8G8B8" hfov="2.094395102" baseline="0.08" focal_length="184.7520861">
-        <origin xyz="0.09 0.0 -0.05" rpy="0 0 0"/>
-    </xacro:generic_stereo_camera>
-    <!-- torch -->
-    <joint name="$torch_joint" type="fixed">
-        <origin xyz="0.06 0.0 0.05" rpy="0 0 0"/>
-        <parent link="link06"/>
-        <child link="torch_frame"/>
-    </joint>
-    <link name="torch_frame">
+    <xacro:if value="$(optenv SPOT_VELODYNE 0)">
+      <!-- Use the Velodyne macro for the actual sensor -->
+      <xacro:include filename="$(find velodyne_description)/urdf/VLP-16.urdf.xacro" />
+      <xacro:VLP-16 parent="lidar_mount">
+        <origin xyz="$(optenv SPOT_VELODYNE_XYZ 0 0 0)" rpy="$(optenv SPOT_VELODYNE_RPY 0 0 0)" />
+      </xacro:VLP-16>
+      <!-- Add the protective cage -->
+      <link name="velodyne_cage">
         <visual>
-            <origin xyz="0 0 0" rpy="0 ${-M_PI/2.0} ${M_PI}" />
-            <geometry>
-                <mesh filename="package://spot_description/meshes/torch.stl" scale="1 1 1"/>
-            </geometry>
+          <geometry>
+            <mesh filename="package://spot_description/meshes/velodyne_cage.stl" scale="0.001 0.001 0.001" />
+          </geometry>
+          <origin xyz="0 0 0" rpy="0 0 0" />
+          <material name="black" />
         </visual>
-    </link>
+        <collision>
+          <geometry>
+            <mesh filename="package://spot_description/meshes/velodyne_cage.stl" scale="0.001 0.001 0.001" />
+          </geometry>
+          <origin xyz="0 0 0" rpy="0 0 0" />
+        </collision>
+      </link>
+      <joint name="velodyne_cage_joint" type="fixed">
+        <parent link="lidar_mount" />
+        <child link="velodyne_cage" />
+        <origin xyz="$(optenv SPOT_VELODYNE_XYZ 0 0 0)" rpy="$(optenv SPOT_VELODYNE_RPY 0 0 0)" />
+      </joint>
+    </xacro:if>
+  </xacro:if>
+  <xacro:if value="$(optenv SPOT_ARM 0)">
+    <xacro:include filename="$(find spot_description)/urdf/spot_arm.xacro" />
+  </xacro:if>
 </robot>

File: src/simulation/robot/spot_description/urdf/spot.urdf.xacro (robot description, xacro)
@@ -1,5 +1,4 @@
 <?xml version="1.0" ?>
 <robot name="spot" xmlns:xacro="http://www.ros.org/wiki/xacro">
-    <xacro:include filename="$(find spot_description)/urdf/constants.urdf.xacro" />
     <link name="body">
         <visual>
@@ -13,10 +12,4 @@
             </geometry>
         </collision>
-        <inertial>
-            <mass value="${base_mass}"/>
-            <inertia ixx="${(1/12) * base_mass * (base_width * base_width + base_height * base_height)}" ixy="0.0" ixz="0.0"
-                        iyy="${(1/12) * base_mass * (base_length * base_length + base_height * base_height)}" iyz="0.0"
-                        izz="${(1/12) * base_mass * (base_length * base_length + base_width * base_width)}" />
-        </inertial>
     </link>
     <link name="base_link"/>
@@ -32,4 +25,10 @@
         <child link="front_rail" />
     </joint>
+    <link name="real_front_rail"/>
+    <joint name="real_front_rail_joint" type="fixed">
+        <origin xyz="0.2075 0 0.0805" rpy="0 0 0" />
+        <parent link="body" />
+        <child link="real_front_rail" />
+    </joint>
     <link name="rear_rail"/>
     <joint name="rear_rail_joint" type="fixed">
@@ -38,29 +37,241 @@
         <child link="rear_rail" />
     </joint>
+    <link name="real_rear_rail"/>
+    <joint name="real_rear_rail_joint" type="fixed">
+        <origin xyz="-0.415 0 0" rpy="0 0 0" />
+        <parent link="real_front_rail" />
+        <child link="real_rear_rail" />
+    </joint>
+    <link name="front_left_hip">
+        <visual>
+            <geometry>
+                <mesh filename="package://spot_description/meshes/front_left_hip.dae" />
+            </geometry>
+        </visual>
+        <collision>
+            <geometry>
+                <mesh filename="package://spot_description/meshes/front_left_hip_collision.stl" />
+            </geometry>
+        </collision>
+    </link>
+    <joint name="front_left_hip_x" type="revolute">
+        <origin xyz="0.29785 0.05500 0.00000" rpy="0 0 0" />
+        <axis xyz="1 0 0" />
+        <parent link="body" />
+        <child link="front_left_hip" />
+        <limit effort="1000" velocity="1000.00" lower="-0.78539816339744827899" upper="0.78539816339744827899" />
+    </joint>
+    <link name="front_left_upper_leg">
+        <visual>
+            <geometry>
+                <mesh filename="package://spot_description/meshes/front_left_upper_leg.dae" />
+            </geometry>
+        </visual>
+        <collision>
+            <geometry>
+                <mesh filename="package://spot_description/meshes/front_left_upper_leg_collision.stl" />
+            </geometry>
+        </collision>
+    </link>
+    <joint name="front_left_hip_y" type="revolute">
+        <origin xyz="0.0 0.110945 0.0" rpy="0 0 0" />
+        <axis xyz="0 1 0" />
+        <parent link="front_left_hip" />
+        <child link="front_left_upper_leg" />
+        <limit effort="1000" velocity="1000.00" lower="-0.89884456477707963539" upper="2.2951079663725435509" />
+    </joint>
+    <link name="front_left_lower_leg">
+        <visual>
+            <geometry>
+                <mesh filename="package://spot_description/meshes/front_left_lower_leg.dae" />
+            </geometry>
+        </visual>
+        <collision>
+            <geometry>
+                <mesh filename="package://spot_description/meshes/front_left_lower_leg_collision.stl" />
+            </geometry>
+        </collision>
+    </link>
+    <joint name="front_left_knee" type="revolute">
+        <origin xyz="0.025 0.000 -0.3205" rpy="0 0 0" />
+        <axis xyz="0 1 0" />
+        <parent link="front_left_upper_leg" />
+        <child link="front_left_lower_leg" />
+        <limit effort="1000" velocity="1000.00" lower="-2.7929" upper="-0.254801" />
+    </joint>
+    <link name="front_right_hip">
+        <visual>
+            <geometry>
+                <mesh filename="package://spot_description/meshes/front_right_hip.dae" />
+            </geometry>
+        </visual>
+        <collision>
+            <geometry>
+                <mesh filename="package://spot_description/meshes/front_right_hip_collision.stl" />
+            </geometry>
+        </collision>
+    </link>
+    <joint name="front_right_hip_x" type="revolute">
+        <origin xyz="0.29785 -0.05500 0.00000" rpy="0 0 0" />
+        <axis xyz="1 0 0" />
+        <parent link="body" />
+        <child link="front_right_hip" />
+        <limit effort="1000" velocity="1000.00" lower="-0.78539816339744827899" upper="0.78539816339744827899" />
+    </joint>
+    <link name="front_right_upper_leg">
+        <visual>
+            <geometry>
+                <mesh filename="package://spot_description/meshes/front_right_upper_leg.dae" />
+            </geometry>
+        </visual>
+        <collision>
+            <geometry>
+                <mesh filename="package://spot_description/meshes/front_right_upper_leg_collision.stl" />
+            </geometry>
+        </collision>
+    </link>
+    <joint name="front_right_hip_y" type="revolute">
+        <origin xyz="0.0 -0.110945 0.0" rpy="0 0 0" />
+        <axis xyz="0 1 0" />
+        <parent link="front_right_hip" />
+        <child link="front_right_upper_leg" />
+        <limit effort="1000" velocity="1000.00" lower="-0.89884456477707963539" upper="2.2951079663725435509" />
+    </joint>
+    <link name="front_right_lower_leg">
+        <visual>
+            <geometry>
+                <mesh filename="package://spot_description/meshes/front_right_lower_leg.dae" />
+            </geometry>
+        </visual>
+        <collision>
+            <geometry>
+                <mesh filename="package://spot_description/meshes/front_right_lower_leg_collision.stl" />
+            </geometry>
+        </collision>
+    </link>
+    <joint name="front_right_knee" type="revolute">
+        <origin xyz="0.025 0.000 -0.3205" rpy="0 0 0" />
+        <axis xyz="0 1 0" />
+        <parent link="front_right_upper_leg" />
+        <child link="front_right_lower_leg" />
+        <limit effort="1000" velocity="1000.00" lower="-2.7929" upper="-0.247563" />
+    </joint>
+    <link name="rear_left_hip">
+        <visual>
+            <geometry>
+                <mesh filename="package://spot_description/meshes/rear_left_hip.dae" />
+            </geometry>
+        </visual>
+        <collision>
+            <geometry>
+                <mesh filename="package://spot_description/meshes/rear_left_hip_collision.stl" />
+            </geometry>
+        </collision>
+    </link>
+    <joint name="rear_left_hip_x" type="revolute">
+        <origin xyz="-0.29785 0.05500 0.00000" rpy="0 0 0" />
+        <axis xyz="1 0 0" />
+        <parent link="body" />
+        <child link="rear_left_hip" />
+        <limit effort="1000" velocity="1000.00" lower="-0.78539816339744827899" upper="0.78539816339744827899" />
+    </joint>
+    <link name="rear_left_upper_leg">
+        <visual>
+            <geometry>
+                <mesh filename="package://spot_description/meshes/rear_left_upper_leg.dae" />
+            </geometry>
+        </visual>
+        <collision>
+            <geometry>
+                <mesh filename="package://spot_description/meshes/rear_left_upper_leg_collision.stl" />
+            </geometry>
+        </collision>
+    </link>
+    <joint name="rear_left_hip_y" type="revolute">
+        <origin xyz="0.0 0.110945 0.0" rpy="0 0 0" />
+        <axis xyz="0 1 0" />
+        <parent link="rear_left_hip" />
+        <child link="rear_left_upper_leg" />
+        <limit effort="1000" velocity="1000.00" lower="-0.89884456477707963539" upper="2.2951079663725435509" />
+    </joint>
+    <link name="rear_left_lower_leg">
+        <visual>
+            <geometry>
+                <mesh filename="package://spot_description/meshes/rear_left_lower_leg.dae" />
+            </geometry>
+        </visual>
+        <collision>
+            <geometry>
+                <mesh filename="package://spot_description/meshes/rear_left_lower_leg_collision.stl" />
+            </geometry>
+        </collision>
+    </link>
+    <joint name="rear_left_knee" type="revolute">
+        <origin xyz="0.025 0.000 -0.3205" rpy="0 0 0" />
+        <axis xyz="0 1 0" />
+        <parent link="rear_left_upper_leg" />
+        <child link="rear_left_lower_leg" />
+        <limit effort="1000" velocity="1000.00" lower="-2.7929" upper="-0.267153" />
+    </joint>
+    <link name="rear_right_hip">
+        <visual>
+            <geometry>
+                <mesh filename="package://spot_description/meshes/rear_right_hip.dae" />
+            </geometry>
+        </visual>
+        <collision>
+            <geometry>
+                <mesh filename="package://spot_description/meshes/rear_right_hip_collision.stl" />
+            </geometry>
+        </collision>
+    </link>
+    <joint name="rear_right_hip_x" type="revolute">
+        <origin xyz="-0.29785 -0.05500 0.00000" rpy="0 0 0" />
+        <axis xyz="1 0 0" />
+        <parent link="body" />
+        <child link="rear_right_hip" />
+        <limit effort="1000" velocity="1000.00" lower="-0.78539816339744827899" upper="0.78539816339744827899" />
+    </joint>
+    <link name="rear_right_upper_leg">
+        <visual>
+            <geometry>
+                <mesh filename="package://spot_description/meshes/rear_right_upper_leg.dae" />
+            </geometry>
+        </visual>
+        <collision>
+            <geometry>
+                <mesh filename="package://spot_description/meshes/rear_right_upper_leg_collision.stl" />
+            </geometry>
+        </collision>
+    </link>
+    <joint name="rear_right_hip_y" type="revolute">
+        <origin xyz="0.0 -0.110945 0.0" rpy="0 0 0" />
+        <axis xyz="0 1 0" />
+        <parent link="rear_right_hip" />
+        <child link="rear_right_upper_leg" />
+        <limit effort="1000" velocity="1000.00" lower="-0.89884456477707963539" upper="2.2951079663725435509" />
+    </joint>
+    <link name="rear_right_lower_leg">
+        <visual>
+            <geometry>
+                <mesh filename="package://spot_description/meshes/rear_right_lower_leg.dae" />
+            </geometry>
+        </visual>
+        <collision>
+            <geometry>
+                <mesh filename="package://spot_description/meshes/rear_right_lower_leg_collision.stl" />
+            </geometry>
+        </collision>
+    </link>
+    <joint name="rear_right_knee" type="revolute">
+        <origin xyz="0.025 0.000 -0.3205" rpy="0 0 0" />
+        <axis xyz="0 1 0" />
+        <parent link="rear_right_upper_leg" />
+        <child link="rear_right_lower_leg" />
+        <limit effort="1000" velocity="1000.00" lower="-2.7929" upper="-0.257725" />
+    </joint>
+    <!-- Standard accessories. -->
+    <xacro:include filename="$(find spot_description)/urdf/accessories.urdf.xacro" />
     <!-- Optional custom includes. -->
     <xacro:include filename="$(optenv SPOT_URDF_EXTRAS empty.urdf)" />
-    <xacro:include filename="$(find spot_description)/urdf/accessories.urdf.xacro" />
-    <xacro:include filename="$(find spot_description)/urdf/spot_leg.urdf.xacro" />
-    <xacro:include filename="$(find spot_description)/urdf/arm.xacro" />
-    <xacro:spot_leg leg_name="front_left"/>
-    <xacro:spot_leg leg_name="front_right"/>
-    <xacro:spot_leg leg_name="rear_left"/>
-    <xacro:spot_leg leg_name="rear_right"/>
-   <gazebo>
-      <plugin name="p3d_base_controller" filename="libgazebo_ros_p3d.so">
-            <alwaysOn>true</alwaysOn>
-            <updateRate>10.0</updateRate>
-            <bodyName>base_link</bodyName>
-            <topicName>odom/ground_truth</topicName>
-            <gaussianNoise>0.01</gaussianNoise>
-            <frameName>world</frameName>
-            <xyzOffsets>0 0 0</xyzOffsets>
-            <rpyOffsets>0 0 0</rpyOffsets>
-        </plugin>
-    </gazebo>
-    <gazebo>
-        <plugin name="gazebo_ros_control" filename="libgazebo_ros_control.so">
-            <legacyModeNS>true</legacyModeNS>
-        </plugin>
-    </gazebo>
 </robot>
